File: Hardware/MOSFET_PowerControlKit.brd (EAGLE design)
At the start: 29.2 x 10.2 mm, 11 parts, among them Q1 IRF

Commit message: Added measurements and version #
Parts:
- removed JP7: LOGO-SFESK, SparkFun:SFE-LOGO-FLAME
- added LOGO2: SFE_LOGO_FLAME.1_INCH, SparkFun-Aesthetics:SFE_LOGO_FLAME_.1
- moved LOGO1 0.34 mm to (8.18, 2.41), turned to 270 degrees
Other:
- board text added: "V11"
Changed lines of the file:
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@@
 <layer number="45" name="Holes" color="7" fill="1" visible="yes" active="yes"/>
 <layer number="46" name="Milling" color="3" fill="1" visible="no" active="yes"/>
-<layer number="47" name="Measures" color="7" fill="1" visible="no" active="yes"/>
+<layer number="47" name="Measures" color="7" fill="1" visible="yes" active="yes"/>
 <layer number="48" name="Document" color="7" fill="1" visible="no" active="yes"/>
-<layer number="49" name="Reference" color="7" fill="1" visible="yes" active="yes"/>
+<layer number="49" name="Reference" color="7" fill="1" visible="no" active="yes"/>
 <layer number="50" name="dxf" color="7" fill="1" visible="no" active="yes"/>
 <layer number="51" name="tDocu" color="6" fill="1" visible="yes" active="yes"/>
@@
 <text x="18.4404" y="-16.5862" size="1.778" layer="51">N. Seidle</text>
 <text x="-0.4064" y="-19.2024" size="1.778" layer="51">Revised by: P. Alberts</text>
+<text x="25.527" y="8.636" size="0.8128" layer="16" font="vector" ratio="15" rot="MR0">V11</text>
+<dimension x1="-2.54" y1="16.51" x2="26.67" y2="16.51" x3="12.065" y3="17.78" textsize="1.778" textratio="15" layer="47"/>
+<dimension x1="-10.16" y1="0" x2="-10.16" y2="10.16" x3="-11.43" y3="5.08" textsize="1.778" textratio="15" layer="47"/>
 </plain>
 <attributes>
@@
 <attribute name="VALUE" x="14.859" y="6.096" size="0.8128" layer="21" ratio="15" rot="SR270"/>
 </element>
-<element name="JP7" library="SparkFun" package="SFE-LOGO-FLAME" value="LOGO-SFESK" x="6.6548" y="6.2484" rot="MR90"/>
 <element name="JP8" library="SparkFun" package="JST-2-PTH" value="" x="21.59" y="5.08" rot="R270"/>
 <element name="JP2" library="SparkFun" package="JST-3-PTH" value="" x="-2.54" y="5.08" rot="R90"/>
@@
 <element name="JP5" library="SparkFun" package="1X03" value="" x="5.08" y="2.54" rot="R90"/>
 <element name="FRAME1" library="SparkFun-Aesthetics" package="CREATIVE_COMMONS" value="FRAME-LETTER" x="-11.91105625" y="-16.51"/>
-<element name="LOGO1" library="SparkFun-Aesthetics" package="OSHW-LOGO-S" value="OSHW-LOGOS" x="7.9502" y="2.667" rot="MR90"/>
+<element name="LOGO1" library="SparkFun-Aesthetics" package="OSHW-LOGO-S" value="OSHW-LOGOS" x="8.1788" y="2.413" rot="MR270"/>
+<element name="LOGO2" library="SparkFun-Aesthetics" package="SFE_LOGO_FLAME_.1" value="SFE_LOGO_FLAME.1_INCH" x="9.525" y="7.239" rot="MR270"/>
 </elements>
 <signals>

Commit message: Qc checklist fixes
Added max current / voltage to sch
fixed airwire
Parts:
- Q1: value IRF -> RFP30N6LE
Routing:
- net HIGH-CURRENT: track 14.0 -> 13.2 mm
Other:
- board text added: "Maximum Current is 30A"
Changed lines of the file:
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@@
 <layer number="47" name="Measures" color="7" fill="1" visible="yes" active="yes"/>
 <layer number="48" name="Document" color="7" fill="1" visible="no" active="yes"/>
-<layer number="49" name="Reference" color="7" fill="1" visible="no" active="yes"/>
+<layer number="49" name="Reference" color="7" fill="1" visible="yes" active="yes"/>
 <layer number="50" name="dxf" color="7" fill="1" visible="no" active="yes"/>
 <layer number="51" name="tDocu" color="6" fill="1" visible="yes" active="yes"/>
@@
 <dimension x1="-2.54" y1="16.51" x2="26.67" y2="16.51" x3="12.065" y3="17.78" textsize="1.778" textratio="15" layer="47"/>
 <dimension x1="-10.16" y1="0" x2="-10.16" y2="10.16" x3="-11.43" y3="5.08" textsize="1.778" textratio="15" layer="47"/>
+<text x="19.939" y="8.001" size="1.778" layer="21" font="vector" ratio="15" rot="R90">-</text>
+<text x="19.685" y="0.762" size="1.778" layer="22" font="vector" ratio="15" rot="MR0">+</text>
+<text x="18.415" y="0.762" size="1.778" layer="21" font="vector" ratio="15">+</text>
+<text x="0" y="-5.08" size="1.27" layer="51" font="vector" ratio="10">Maximum Current is 30A</text>
 </plain>
 <attributes>
@@
 </autorouter>
 <elements>
-<element name="Q1" library="SparkFun" package="TO220V" value="IRF" x="11.43" y="5.08" rot="R270"/>
+<element name="Q1" library="SparkFun" package="TO220V" value="RFP30N6LE" x="11.43" y="5.08" rot="R270"/>
 <element name="R1" library="SparkFun" package="AXIAL-0.3" value="10K" x="15.24" y="5.08" smashed="yes" rot="R90">
 <attribute name="NAME" x="13.97" y="2.54" size="0.4064" layer="25" rot="R90"/>
@@
 <wire x1="21.59" y1="6.08" x2="22.844" y2="6.08" width="2.032" layer="1"/>
 <wire x1="22.844" y1="6.08" x2="23.622" y2="6.858" width="2.032" layer="1"/>
-<wire x1="10.5918" y1="5.08" x2="15.621" y2="5.08" width="2.032" layer="1"/>
 <wire x1="15.621" y1="5.08" x2="16.9164" y2="6.3754" width="2.032" layer="1"/>
 <wire x1="16.9164" y1="6.3754" x2="19.0246" y2="6.3754" width="2.032" layer="1"/>
 <wire x1="19.0246" y1="6.3754" x2="19.05" y2="6.35" width="2.032" layer="1"/>
-<wire x1="10.5918" y1="5.08" x2="11.43" y2="5.08" width="0" layer="19" extent="1-1"/>
+<wire x1="15.621" y1="5.08" x2="11.43" y2="5.08" width="1.9304" layer="1"/>
 </signal>
 </signals>

Commit message: More qc checklist changes
Other:
- board text removed: "Maximum Current is 30A"
Changed lines of the file:
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@@
 <layer number="45" name="Holes" color="7" fill="1" visible="yes" active="yes"/>
 <layer number="46" name="Milling" color="3" fill="1" visible="no" active="yes"/>
-<layer number="47" name="Measures" color="7" fill="1" visible="yes" active="yes"/>
+<layer number="47" name="Measures" color="7" fill="1" visible="no" active="yes"/>
 <layer number="48" name="Document" color="7" fill="1" visible="no" active="yes"/>
-<layer number="49" name="Reference" color="7" fill="1" visible="yes" active="yes"/>
+<layer number="49" name="Reference" color="7" fill="1" visible="no" active="yes"/>
 <layer number="50" name="dxf" color="7" fill="1" visible="no" active="yes"/>
 <layer number="51" name="tDocu" color="6" fill="1" visible="yes" active="yes"/>
@@
 <text x="19.685" y="0.762" size="1.778" layer="22" font="vector" ratio="15" rot="MR0">+</text>
 <text x="18.415" y="0.762" size="1.778" layer="21" font="vector" ratio="15">+</text>
-<text x="0" y="-5.08" size="1.27" layer="51" font="vector" ratio="10">Maximum Current is 30A</text>
 </plain>
 <attributes>
